File: kicad/kicad_timer.kicad_sch (KiCad schematic)
At the start: 14 parts, among them J1 USB_C_Receptacle_PowerOnly_6P, U1 CA56-12CGKWA, U2 ATmega328-A, U3 CA56-12CGKWA

Commit message: Improving the pcb
Parts:
- R1, R2, R3: value Resistor -> 1K
- R4, R5: value Resistor -> 5.11 K
- R6: value Resistor -> 1M resistor
- S2, S3: footprint hotswap:Hotswap_MX -> kbd:keyswitch_cherrymx_hotswap_1u
Connections:
- no-connect marks 0 -> 7
Other:
- moved on the sheet: R6, U3
Changed lines of the file:
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@@
 		(color 0 0 0 0)
 	)
+	(no_connect
+		(at 116.84 45.72)
+	)
+	(no_connect
+		(at 77.47 27.94)
+	)
+	(no_connect
+		(at 120.65 68.58)
+	)
+	(no_connect
+		(at 107.95 71.12)
+	)
+	(no_connect
+		(at 107.95 45.72)
+	)
+	(no_connect
+		(at 77.47 35.56)
+	)
+	(no_connect
+		(at 77.47 33.02)
+	)
 	(wire
 		(pts
@@
 	(wire
 		(pts
-			(xy 107.95 38.1) (xy 120.65 38.1)
-		)
-		(stroke
-			(width 0)
-			(type default)
-		)
-	)
-	(wire
-		(pts
-			(xy 107.95 30.48) (xy 120.65 30.48)
+			(xy 107.95 38.1) (xy 116.84 38.1)
+		)
+		(stroke
+			(width 0)
+			(type default)
+		)
+	)
+	(wire
+		(pts
+			(xy 107.95 30.48) (xy 116.84 30.48)
 		)
 		(stroke
@@
 	(wire
 		(pts
-			(xy 107.95 35.56) (xy 120.65 35.56)
+			(xy 107.95 35.56) (xy 116.84 35.56)
 		)
 		(stroke
@@
 	(wire
 		(pts
+			(xy 172.72 43.18) (xy 176.53 43.18)
+		)
+		(stroke
+			(width 0)
+			(type default)
+		)
+	)
+	(wire
+		(pts
 			(xy 107.95 50.8) (xy 120.65 50.8)
 		)
@@
 	(wire
 		(pts
-			(xy 107.95 33.02) (xy 120.65 33.02)
-		)
-		(stroke
-			(width 0)
-			(type default)
-		)
-	)
-	(wire
-		(pts
-			(xy 107.95 40.64) (xy 120.65 40.64)
+			(xy 107.95 33.02) (xy 116.84 33.02)
+		)
+		(stroke
+			(width 0)
+			(type default)
+		)
+	)
+	(wire
+		(pts
+			(xy 107.95 40.64) (xy 116.84 40.64)
 		)
 		(stroke
@@
 	(wire
 		(pts
-			(xy 24.13 123.19) (xy 24.13 125.73)
+			(xy 172.72 40.64) (xy 176.53 40.64)
+		)
+		(stroke
+			(width 0)
+			(type default)
+		)
+	)
+	(wire
+		(pts
+			(xy 24.13 121.92) (xy 24.13 124.46)
 		)
 		(stroke
@@
 	(wire
 		(pts
+			(xy 172.72 45.72) (xy 176.53 45.72)
+		)
+		(stroke
+			(width 0)
+			(type default)
+		)
+	)
+	(wire
+		(pts
 			(xy 48.26 53.34) (xy 50.8 53.34)
 		)
@@
 	(wire
 		(pts
-			(xy 107.95 43.18) (xy 120.65 43.18)
+			(xy 107.95 43.18) (xy 116.84 43.18)
 		)
 		(stroke
@@
 	(wire
 		(pts
+			(xy 172.72 38.1) (xy 176.53 38.1)
+		)
+		(stroke
+			(width 0)
+			(type default)
+		)
+	)
+	(wire
+		(pts
 			(xy 55.88 35.56) (xy 59.69 35.56)
 		)
@@
 	(wire
 		(pts
-			(xy 107.95 27.94) (xy 120.65 27.94)
+			(xy 107.95 27.94) (xy 116.84 27.94)
 		)
 		(stroke
@@
 	(wire
 		(pts
-			(xy 24.13 111.76) (xy 24.13 115.57)
+			(xy 24.13 111.76) (xy 24.13 114.3)
 		)
 		(stroke
@@
 	(global_label "GND"
 		(shape input)
-		(at 24.13 125.73 270)
+		(at 24.13 124.46 270)
 		(fields_autoplaced yes)
 		(effects
@@
 		)
 		(property "Intersheetrefs" "${INTERSHEET_REFS}"
-			(at 24.13 132.5857 90)
+			(at 24.13 131.3157 90)
 			(effects
 				(font
@@
 		(dnp no)
 		(property "Reference" "R1"
-			(at 24.13 44.704 0)
+			(at 24.13 41.91 0)
 			(effects
 				(font
@@
 			)
 		)
-		(property "Value" "Resistor"
-			(at 24.13 36.83 0)
+		(property "Value" "1K"
+			(at 24.13 38.1 0)
 			(effects
 				(font
@@
 			)
 		)
-		(property "Footprint" "hotswap:Hotswap_MX"
+		(property "Footprint" "kbd:keyswitch_cherrymx_hotswap_1u"
 			(at 53.34 55.88 0)
 			(effects
@@
 		(dnp no)
 		(property "Reference" "R2"
-			(at 27.94 44.704 0)
+			(at 27.94 41.91 0)
 			(effects
 				(font
@@
 			)
 		)
-		(property "Value" "Resistor"
-			(at 27.94 36.576 0)
+		(property "Value" "1K"
+			(at 27.94 38.354 0)
 			(effects
 				(font
@@
 			)
 		)
-		(property "Footprint" "hotswap:Hotswap_MX"
+		(property "Footprint" "kbd:keyswitch_cherrymx_hotswap_1u"
 			(at 53.34 44.45 0)
 			(effects
@@
 			)
 		)
-		(property "Value" "Resistor"
+		(property "Value" "5.11 K"
 			(at 44.45 107.696 90)
 			(effects
@@
 	(symbol
 		(lib_id "Keyboard:Placeholder_Resistor")
-		(at 24.13 119.38 270)
+		(at 24.13 118.11 270)
 		(unit 1)
 		(exclude_from_sim no)
@@
 		(dnp no)
 		(property "Reference" "R6"
-			(at 15.24 117.856 90)
-			(effects
-				(font
-					(size 1.27 1.27)
-				)
-				(justify left)
-			)
-		)
-		(property "Value" "Resistor"
-			(at 15.24 120.396 90)
+			(at 19.05 116.84 0)
+			(effects
+				(font
+					(size 1.27 1.27)
+				)
+				(justify left)
+			)
+		)
+		(property "Value" "1M resistor"
+			(at 21.59 113.03 0)
 			(effects
 				(font
@@
 		)
 		(property "Footprint" "Resistor_SMD:R_0201_0603Metric"
-			(at 22.352 119.38 0)
+			(at 22.352 118.11 0)
 			(effects
 				(font
@@
 		)
 		(property "Datasheet" "~"
-			(at 24.13 119.38 90)
+			(at 24.13 118.11 90)
 			(effects
 				(font
@@
 		)
 		(property "Description" "Resistor"
-			(at 24.13 119.38 0)
+			(at 24.13 118.11 0)
 			(effects
 				(font
@@
 			)
 		)
-		(property "Value" "Resistor"
+		(property "Value" "5.11 K"
 			(at 60.96 107.9499 90)
 			(effects
@@
 		(on_board yes)
 		(dnp no)
-		(fields_autoplaced yes)
 		(property "Reference" "R3"
-			(at 31.75 44.958 0)
+			(at 31.75 42.164 0)
 			(effects
 				(font
@@
 			)
 		)
-		(property "Value" "Resistor"
-			(at 31.75 36.83 0)
+		(property "Value" "1K"
+			(at 31.75 38.1 0)
 			(effects
 				(font
@@
 	(symbol
 		(lib_id "Display_Character:CA56-12CGKWA")
-		(at 148.59 35.56 0)
+		(at 144.78 35.56 0)
 		(unit 1)
 		(exclude_from_sim no)
@@
 		(fields_autoplaced yes)
 		(property "Reference" "U3"
-			(at 148.59 17.78 0)
+			(at 144.78 17.78 0)
 			(effects
 				(font
@@
 		)
 		(property "Value" "CA56-12CGKWA"
-			(at 148.59 20.32 0)
+			(at 144.78 20.32 0)
 			(effects
 				(font
@@
 		)
 		(property "Footprint" "Display_7Segment:CA56-12CGKWA"
-			(at 148.59 50.8 0)
+			(at 144.78 50.8 0)
 			(effects
 				(font
@@
 		)
 		(property "Datasheet" "http://www.kingbright.com/attachments/file/psearch/000/00/00/CA56-12CGKWA(Ver.9A).pdf"
-			(at 137.668 34.798 0)
+			(at 133.858 34.798 0)
 			(effects
 				(font
@@
 		)
 		(property "Description" "4 digit 7 segment Green LED, common anode"
-			(at 148.59 35.56 0)
-			(effects
-				(font
+			(at 144.78 35.56 0)
+			(effects
+				(font
